Commit message: [Configuration] Update the joint axis for the hip

File: walker_description/urdf/simple_walker.urdf.xacro (robot description, xacro)
@@ -40,4 +40,5 @@
         <parent link="body" />
         <child link="thigh_left" />
+        <axis xyz="0 1 0" />
         <origin xyz="0 ${-bodyheight} ${-(bodydepth / 2 + shank_length)}" />
         <limit effort="100" lower="-0.5" upper="0.5" velocity="10"/>
@@ -48,4 +49,5 @@
         <parent link="body" />
         <child link="thigh_right" />
+        <axis xyz="0 1 0" />
         <origin xyz="0 ${bodyheight} ${-(bodydepth / 2 + shank_length)}" />
         <limit effort="100" lower="-0.5" upper="0.5" velocity="10"/>

Commit message: [Refactor] Include dummy link with no inertia

File: walker_description/urdf/simple_walker.urdf.xacro (robot description, xacro)
@@ -8,4 +8,6 @@
     <xacro:property name="bodyheight" value="0.3" />
     <xacro:property name="bodydepth" value="0.3" />
+    <link name="base_link">
+    </link>
     <!-- Define the upper portion of the robot -->
     <link name="body">
@@ -35,4 +37,9 @@
     <!-- Include components -->
     <xacro:include filename="$(find walker_description)/urdf/walker_leg.macro.xacro" />
+    <!-- Attach dummy root link to body -->
+    <joint name="base_link_to_body" type="fixed">
+        <parent link="base_link" />
+        <child link="body" />
+    </joint>
     <!-- Instantiate the left leg of the robot -->
     <xacro:walker_leg_macro id="left" />
@@ -55,5 +62,5 @@
     <!-- Include hardware configuration for ros2_control -->
     <xacro:include filename="$(find walker_description)/urdf/ros2_control/simple_walker.ros2_control.xacro" />
-    <xacro:walker_ros2_control name="walker" plugin="fake_components/GenericSystem" />
+    <xacro:walker_ros2_control name="walker" plugin="gazebo_ros2_control/GazeboSystem" />
     <!-- Specify the Gazebo plugin for interfacing with ros2_control -->
     <gazebo>

Commit message: [Configuration] Update inertial matrix in robot description

File: walker_description/urdf/simple_walker.urdf.xacro (robot description, xacro)
@@ -25,12 +25,12 @@
         </collision>
         <inertial>
-            <mass value="${massbody}" />
+            <mass value="1" />
             <inertia
-                ixx="${1/12 * massbody * (bodyheight*bodyheight + bodydepth*bodydepth)}"
-                iyy="${1/12 * massbody * (bodywidth*bodywidth + bodydepth*bodydepth)}"
-                izz="${1/12 * massbody * (bodyheight*bodyheight + bodywidth*bodywidth)}"
+                ixx="1e-1"
                 ixy="0"
                 ixz="0"
-                iyz="0" />
+                iyy="1e-1"
+                iyz="0"
+                izz="1e-1" />
         </inertial>
     </link>

File: walker_description/urdf/walker_leg.macro.xacro (robot description, xacro)
@@ -28,10 +28,10 @@
             <mass value="${thigh_mass}"/>
             <inertia
-                ixx="1e-3"
+                ixx="1e-1"
                 ixy="0"
                 ixz="0"
-                iyy="1e-3"
+                iyy="1e-1"
                 iyz="0"
-                izz="1e-3"/>
+                izz="1e-1" />
         </inertial>
         </link>
@@ -53,10 +53,10 @@
                 <mass value="${shank_mass}"/>
                 <inertia
-                ixx="1e-3"
-                ixy="0"
-                ixz="0"
-                iyy="1e-3"
-                iyz="0"
-                izz="1e-3"/>
+                    ixx="1e-1"
+                    ixy="0"
+                    ixz="0"
+                    iyy="1e-1"
+                    iyz="0"
+                    izz="1e-1" />
                 <origin rpy="0 0 0" xyz="0 0 ${-shank_length/2-knee_joint_radius}"/>
             </inertial>
@@ -89,10 +89,10 @@
                 <mass value="${foot_mass}"/>
                 <inertia
-                ixx="1e-3"
-                ixy="0"
-                ixz="0"
-                iyy="1e-3"
-                iyz="0"
-                izz="1e-3"/>
+                    ixx="1e-1"
+                    ixy="0"
+                    ixz="0"
+                    iyy="1e-1"
+                    iyz="0"
+                    izz="1e-1" />
                 <origin xyz="${(foot_length/2-0.05)} 0 ${-ankle_joint_radius-foot_height/2}"/>
             </inertial>
